Commit message: indoor env improved

File: plugins/urdf/quadrotor_simple_controller.urdf.xacro (robot description, xacro)
@@ -22,8 +22,8 @@
         <velocityXYProportionalGain>5.0</velocityXYProportionalGain>
         <velocityXYDifferentialGain>1.0</velocityXYDifferentialGain>
-        <velocityXYLimit>2</velocityXYLimit>
+        <velocityXYLimit>10</velocityXYLimit>
         <velocityZProportionalGain>5.0</velocityZProportionalGain>
         <velocityZDifferentialGain>1.0</velocityZDifferentialGain>
-        <velocityZLimit>0.5</velocityZLimit>
+        <velocityZLimit>2.5</velocityZLimit>
         <maxForce>30</maxForce>
         <motionSmallNoise>0.05</motionSmallNoise>

File: worlds/xacro/imav_indoor.world.xacro (robot description, xacro)
@@ -11,4 +11,7 @@
     <xacro:gui_/>
     <xacro:scn amb="0.4 0.4 0.4 1" backg="0.7 0.7 0.7 1"/>
+    <!--
+    <xacro:scn amb="0.4 0.4 0.4 1" backg="${53/255} ${147/255} ${37/255} 1"/>
+    -->
     <xacro:zone name="takoff_landing" 	offset="0"	 				width="${width}" length="${length1}" color="${22/255}  ${176/255} ${37/255}"/>
     <xacro:zone name="obstacle" 	offset="${length1/2+length2/2}" 		width="${width}" length="${length2}" color="${188/255} ${53/255}  ${53/255}"/>
@@ -16,5 +19,11 @@
     <xacro:wall_obstacle w_s="0.5" w_b="1" w_t="0.5" offset="${length1/4}" width="${width}" height="3"/>
     <xacro:wall_brand w="${length1+length2+length3}" h="${3*3}"	l="0.2" x="${length1/2+length2/2}" y="${width*2}"	z="${3*3/2}"/>
-    <xacro:poles h="3" r="0.25" w="${width}" l="${length2}" x="${length1/2+length2/2}" y="0"/>
+    <xacro:poles2 h="3" r="0.25" w="${width}" l="${length2/2}" x="${length1/2+length2/4}" y="0"/>
+    <!--
+    <xacro:trees w="${width}" l="${length2/2}" x="${length1/2+3*length2/4}" y="0"/>
+    <xacro:bushes w="${width}" l="${length2/2}" x="${length1/2+3*length2/4}" y="0"/>
+    -->
+    <xacro:helipad_static size="0.5 0.5 0.01" x="1"  y="1"  z="0.1"/>
+    <xacro:helipad_mobile size="0.5 0.5 0.01" x="-1" y="-1" z="0.1" r="1" v="1"/>
   </world>
 </sdf>

File: worlds/xacro/macros.urdf.xacro (robot description, xacro)
@@ -52,5 +52,5 @@
     <light name="sun" type="directional">
       <cast_shadows>1</cast_shadows>
-      <pose>0 0 10 0 -0 0</pose>
+      <pose>0 10 0 0 0 -${pi/2}</pose>
       <diffuse>0.8 0.8 0.8 1</diffuse>
       <specular>0.2 0.2 0.2 1</specular>
@@ -208,4 +208,50 @@
       </visual>
   </xacro:macro>
+  <xacro:macro name="pole2" params="h r">
+    <static>true</static>
+    <link name="pole_link">
+      <collision name="pole_collision">
+	<geometry>
+	  <cylinder>
+	    <radius>${r}</radius>
+	    <length>${h}</length>
+	  </cylinder>
+	</geometry>
+	<surface>
+	  <contact>
+	    <collide_bitmask>0x02</collide_bitmask>
+	  </contact>
+	</surface>
+      </collision>
+      <visual name="pole_visual">
+	<geometry>
+	  <cylinder>
+	    <radius>${r}</radius>
+	    <length>${h}</length>
+	  </cylinder>
+	</geometry>
+	<material>
+	  <script>
+	    <name>Gazebo/Bricks</name>
+	  </script>
+	</material>
+      </visual>
+    </link>
+  </xacro:macro>
+  <xacro:macro name="poles2" params="h r w l x y">
+    <population name="pole_population">
+      <model name="pole">
+	<xacro:pole2 h="${h}" r="${r}"/>
+      </model>
+      <pose>${x} ${y} ${h/2} 0 0 0</pose>
+      <box>
+        <size>${l} ${w} 0.1</size>
+      </box>
+      <model_count>20</model_count>
+      <distribution>
+        <type>uniform</type>
+      </distribution>
+    </population>
+  </xacro:macro>
   <xacro:macro name="poles" params="h r w l x y">
     <model name="poles">
@@ -227,3 +273,98 @@
     </model>
   </xacro:macro>
+  <xacro:macro name="trees" params="w l x y">
+    <population name="pole_population">
+      <model name="pole">
+	<include>
+          <static>true</static>
+          <uri>model://meshes/tree.dae</uri>
+        </include>
+      </model>
+      <pose>${x} ${y} 0 0 0</pose>
+      <box>
+        <size>${l} ${w} 0.1</size>
+      </box>
+      <model_count>10</model_count>
+      <distribution>
+        <type>uniform</type>
+      </distribution>
+    </population>
+  </xacro:macro>
+  <xacro:macro name="bushes" params="w l x y">
+    <population name="pole_population">
+      <model name="pole">
+	<include>
+          <static>true</static>
+          <uri>model://meshes/bush.dae</uri>
+        </include>
+      </model>
+      <pose>${x} ${y} 0 0 0 0</pose>
+      <box>
+        <size>${l} ${w} 0.1</size>
+      </box>
+      <model_count>10</model_count>
+      <distribution>
+        <type>uniform</type>
+      </distribution>
+    </population>
+  </xacro:macro>
+  <xacro:macro name="helipad" params="size x y z">
+      <link name="helipad_link">
+	<pose>${x} ${y} ${z} 0 0 0</pose>
+	<inertial>
+	  <mass>10</mass>
+	</inertial>
+	<collision name="wall_brand_collision">
+	  <geometry>
+	    <box>
+	      <size>${size}</size>
+	    </box>
+	  </geometry>
+	  <surface>
+	    <contact>
+	      <collide_bitmask>0x02</collide_bitmask>
+	    </contact>
+	  </surface>
+	</collision>
+	<visual name="helipad_visual">
+	  <geometry>
+	    <box>
+	      <size>${size}</size>
+	    </box>
+	  </geometry>
+	  <material>
+	    <script>
+	      <uri>file://$(find imav_2017)/worlds/xacro/custom.material</uri>
+	      <name>Helipad</name>
+	    </script>
+	  </material>
+	</visual>
+      </link>
+  </xacro:macro>
+  <xacro:macro name="helipad_static" params="size x y z">
+    <model name="helipad_static">
+      <static>true</static>
+      <xacro:helipad size="${size}" x="${x+1}" y="${y}" z="${z}"/>
+    </model>
+  </xacro:macro>
+  <xacro:macro name="helipad_mobile" params="size x y z r v">
+    <model name="helipad_mobile">
+      <pose>${x} ${y} ${z} 0 0 0</pose>
+      <joint name="helipad_joint" type="revolute">
+	<pose>${x} ${y} ${z} 0 0 0</pose>
+	<parent>world</parent>
+	<child>helipad_link</child>
+	<axis>
+	  <xyz>0 0 1</xyz>
+	</axis>
+	<physics>
+	  <ode>
+	    <velocity>${v}</velocity>
+	    <max_force>1000</max_force>
+	  </ode>
+	</physics>
+      </joint>
+      <xacro:helipad size="${size}" x="${1}" y="0" z="0"/>
+    </model>
+  </xacro:macro>
 </my_macros>
