Commit message: Working stage

File: plugins/urdf/quadrotor_plugins.urdf.xacro (robot description, xacro)
@@ -1,4 +1,4 @@
 <?xml version="1.0"?>
-<robot xmlns:xacro="http://playerstage.sourceforge.net/gazebo/xmlschema/#interface">
+<robot xmlns:xacro="http://wiki.ros.org/xacro" >
   <xacro:include filename="$(find imav_2017)/plugins/urdf/quadrotor_sensors.urdf.xacro" />
   <xacro:include filename="$(find imav_2017)/plugins/urdf/quadrotor_simple_controller.urdf.xacro" />

File: plugins/urdf/quadrotor_sensors.urdf.xacro (robot description, xacro)
@@ -1,8 +1,4 @@
 <?xml version="1.0"?>
-<robot xmlns:sensor="http://playerstage.sourceforge.net/gazebo/xmlschema/#sensor"
-xmlns:controller="http://playerstage.sourceforge.net/gazebo/xmlschema/#controller"
-xmlns:interface="http://playerstage.sourceforge.net/gazebo/xmlschema/#interface"
-xmlns:xacro="http://playerstage.sourceforge.net/gazebo/xmlschema/#interface"
->
+<robot xmlns:xacro="http://wiki.ros.org/xacro" >
   <!-- Quadrotor Sensor Plugins
         <frameId>ardrone_base_link</frameId>

File: plugins/urdf/quadrotor_simple_controller.urdf.xacro (robot description, xacro)
@@ -1,7 +1,4 @@
 <?xml version="1.0"?>
-<robot
-xmlns:controller="http://playerstage.sourceforge.net/gazebo/xmlschema/#controller"
-xmlns:xacro="http://playerstage.sourceforge.net/gazebo/xmlschema/#interface"
->
+<robot xmlns:xacro="http://wiki.ros.org/xacro" >
   <!-- Quadrotor Simple Controller Plugin -->
   <xacro:macro name="quadrotor_controller">

File: urdf/quadrotor_base.urdf.xacro (robot description, xacro)
@@ -27,10 +27,4 @@
       </collision>
     </link>
-    <!--
-    <gazebo reference="base_link">
-      <turnGravityOff>false</turnGravityOff>
-    </gazebo>
-    -->
-    <!-- Gazebo Plugins -->
     <quadrotor_plugins/>
   </xacro:macro>

File: urdf/quadrotor_sensors.urdf.xacro (robot description, xacro)
@@ -1,4 +1,4 @@
 <?xml version="1.0"?>
-<robot name="quadrotor_hokuyo_utm30lx" xmlns:xacro="http://www.ros.org/wiki/xacro">
+<robot name="quadrotor_hokuyo_utm30lx" xmlns:xacro="http://wiki.ros.org/xacro" >
     <xacro:property name="M_PI" value="3.1415926535897931" />
     <!-- Included URDF Files -->

File: urdf/sensors/generic_camera.urdf.xacro (robot description, xacro)
@@ -1,8 +1,4 @@
 <?xml version="1.0"?>
-<robot xmlns:sensor="http://playerstage.sourceforge.net/gazebo/xmlschema/#sensor"
-xmlns:controller="http://playerstage.sourceforge.net/gazebo/xmlschema/#controller"
-xmlns:interface="http://playerstage.sourceforge.net/gazebo/xmlschema/#interface"
-  xmlns:xacro="http://playerstage.sourceforge.net/gazebo/xmlschema/#interface"
-  >
+<robot xmlns:xacro="http://wiki.ros.org/xacro">
     <xacro:property name="M_PI" value="3.1415926535897931" />
     <xacro:macro name="generic_camera" params="name sim_name parent *origin update_rate res_x res_y image_format hfov">

File: urdf/sensors/hokuyo_utm30lx.urdf.xacro (robot description, xacro)
@@ -1,8 +1,4 @@
 <?xml version="1.0"?>
-<robot xmlns:sensor="http://playerstage.sourceforge.net/gazebo/xmlschema/#sensor"
-xmlns:controller="http://playerstage.sourceforge.net/gazebo/xmlschema/#controller"
-xmlns:interface="http://playerstage.sourceforge.net/gazebo/xmlschema/#interface"
-  xmlns:xacro="http://ros.org/wiki/xacro"
-  >
+<robot xmlns:xacro="http://wiki.ros.org/xacro" >
     <xacro:macro name="hokuyo_utm30lx" params="name parent *origin ros_topic update_rate ray_count min_angle max_angle">
       <joint name="${name}_joint" type="fixed">

File: urdf/sensors/sonar_sensor.urdf.xacro (robot description, xacro)
@@ -1,11 +1,4 @@
 <?xml version="1.0"?>
-<robot xmlns:sensor="http://playerstage.sourceforge.net/gazebo/xmlschema/#sensor"
-xmlns:controller="http://playerstage.sourceforge.net/gazebo/xmlschema/#controller"
-xmlns:interface="http://playerstage.sourceforge.net/gazebo/xmlschema/#interface"
-xmlns:xacro="http://playerstage.sourceforge.net/gazebo/xmlschema/#interface"
->
-<!--
-	xmlns:xacro="http://ros.org/wiki/xacro"
--->
+<robot xmlns:xacro="http://wiki.ros.org/xacro" >
   <xacro:macro name="sonar_sensor" params="name parent *origin ros_topic update_rate min_range max_range field_of_view ray_count">
     <joint name="${name}_joint" type="fixed">

File: worlds/xacro/imav_indoor.world.xacro (robot description, xacro)
@@ -19,5 +19,5 @@
     <xacro:wall_obstacle w_s="0.5" w_b="1" w_t="0.5" offset="${length1/4}" width="${width}" height="3"/>
     <xacro:wall_brand w="${length1+length2+length3}" h="${3*3}"	l="0.2" x="${length1/2+length2/2}" y="${width*2}"	z="${3*3/2}"/>
-    <xacro:poles2 h="3" r="0.25" w="${width}" l="${length2/2}" x="${length1/2+length2/4}" y="0"/>
+    <xacro:poles2 h="3" r="0.25" w="${width}" l="${length2}" x="${length1/2+length2/2}" y="0" num="50"/>
     <!--
     <xacro:trees w="${width}" l="${length2/2}" x="${length1/2+3*length2/4}" y="0"/>

File: worlds/xacro/macros.urdf.xacro (robot description, xacro)
@@ -239,5 +239,5 @@
     </link>
   </xacro:macro>
-  <xacro:macro name="poles2" params="h r w l x y">
+  <xacro:macro name="poles2" params="h r w l x y num">
     <population name="pole_population">
       <model name="pole">
@@ -248,7 +248,7 @@
         <size>${l} ${w} 0.1</size>
       </box>
-      <model_count>20</model_count>
+      <model_count>${num}</model_count>
       <distribution>
-        <type>uniform</type>
+        <type>random</type>
       </distribution>
     </population>
