Commit message: Kind-of working stage

File: urdf/sensors/hokuyo_utm30lx.urdf.xacro (robot description, xacro)
@@ -7,5 +7,5 @@
 	<child link="${name}_frame"/>
       </joint>
-<link name="${name}_frame">
+      <link name="${name}_frame">
 	<inertial>
 	  <mass value="0.001" />
@@ -26,28 +26,28 @@
         </geometry>
 	</collision>
-</link>
-  <gazebo reference="${name}_frame">
-    <sensor:ray name="${name}">
-    <rayCount>${ray_count}</rayCount>
-    <rangeCount>${ray_count}</rangeCount>
-        <laserCount>1</laserCount>
-        <origin>0.0 0.0 0.0</origin>
-        <displayRays>false</displayRays>
-        <minAngle>${min_angle}</minAngle>
-        <maxAngle>${max_angle}</maxAngle>
-        <minRange>0.08</minRange>
-        <maxRange>30.0</maxRange>
-        <resRange>0.01</resRange>
-        <updateRate>${update_rate}</updateRate>
-        <controller:gazebo_ros_laser name="gazebo_ros_${name}_controller" plugin="libgazebo_ros_laser.so">
-          <gaussianNoise>0.005</gaussianNoise>
-          <alwaysOn>true</alwaysOn>
-          <updateRate>${update_rate}</updateRate>
-          <topicName>${ros_topic}</topicName>
-          <frameName>${name}_frame</frameName>
-          <interface:laser name="gazebo_ros_${name}_iface" />
-        </controller:gazebo_ros_laser>
-      </sensor:ray>
-    </gazebo>
+      </link>
+      <gazebo reference="${name}_frame">
+	<sensor:ray name="${name}">
+	  <rayCount>${ray_count}</rayCount>
+	  <rangeCount>${ray_count}</rangeCount>
+	  <laserCount>1</laserCount>
+	  <origin>0.0 0.0 0.0</origin>
+	  <displayRays>false</displayRays>
+	  <minAngle>${min_angle}</minAngle>
+	  <maxAngle>${max_angle}</maxAngle>
+	  <minRange>0.08</minRange>
+	  <maxRange>30.0</maxRange>
+	  <resRange>0.01</resRange>
+	  <updateRate>${update_rate}</updateRate>
+	  <controller:gazebo_ros_laser name="gazebo_ros_${name}_controller" plugin="libgazebo_ros_laser.so">
+	    <gaussianNoise>0.005</gaussianNoise>
+	    <alwaysOn>true</alwaysOn>
+	    <updateRate>${update_rate}</updateRate>
+	    <topicName>${ros_topic}</topicName>
+	    <frameName>${name}_frame</frameName>
+	    <interface:laser name="gazebo_ros_${name}_iface" />
+	  </controller:gazebo_ros_laser>
+	</sensor:ray>
+      </gazebo>
     </xacro:macro>
   </robot>
