Commit message: Bottom camera orientation fixed

File: urdf/quadrotor_with_sensors.urdf.xacro (robot description, xacro)
@@ -25,5 +25,5 @@
     <xacro:include filename="$(find imav_2017)/urdf/sensors/generic_camera.urdf.xacro" />
     <xacro:generic_camera name="bottom" sim_name="ardrone" parent="base_link" update_rate="60" res_x="640" res_y="360" image_format="R8G8B8" hfov="${81*M_PI/180}">
-      <origin xyz="0.15 0.0 0.0" rpy="0 -${M_PI/2} 0"/>
+      <origin xyz="0.15 0.0 0.0" rpy="0 ${M_PI/2} 0"/>
     </xacro:generic_camera>
 </robot>

Commit message: Trying to fix hokuyo

File: urdf/quadrotor_with_sensors.urdf.xacro (robot description, xacro)
@@ -17,4 +17,6 @@
     </xacro:hokuyo_utm30lx>
     -->
+    <xacro:include filename="$(find imav_2017)/urdf/sensors/hokuyo_utm30lx.urdf.xacro" />
+    <xacro:hokuyo parent="base_link" ros_topic="scan" update_rate="40" ray_count="1081" min_angle="135" max_angle="-135"/>
     <!-- The following two cameras should be united to one! -->
     <!-- Forward facing camera -->

File: urdf/sensors/hokuyo_utm30lx.urdf.xacro (robot description, xacro)
@@ -1,4 +1,5 @@
 <?xml version="1.0"?>
 <robot xmlns:xacro="http://wiki.ros.org/xacro" >
+    <!--
     <xacro:macro name="hokuyo_utm30lx" params="name parent *origin ros_topic update_rate ray_count min_angle max_angle">
       <joint name="${name}_joint" type="fixed">
@@ -23,5 +24,5 @@
           <geometry>
           <box size="0.058 0.058 0.087" />
-          <!--<mesh filename="package://hector_sensors_description/meshes/hokuyo_utm30lx/hokuyo_utm_30lx.stl"/>-->
+          <mesh filename="package://hector_sensors_description/meshes/hokuyo_utm30lx/hokuyo_utm_30lx.stl"/>
         </geometry>
 	</collision>
@@ -51,3 +52,21 @@
       </gazebo>
     </xacro:macro>
-  </robot>
+    -->
+  <xacro:macro name="hokuyo" params="parent ros_topic update_rate ray_count min_angle max_angle">
+      <include>
+	<uri>model://hokuyo</uri>
+	<pose>0.2 0 0.2 0 0 0</pose>
+      </include>
+      <joint name="hokuyo_joint" type="revolute">
+	<child>hokuyo::link</child>
+	<parent>${parent}</parent>
+	<axis>
+	  <xyz>0 0 1</xyz>
+	  <limit>
+	    <upper>0</upper>
+	    <lower>0</lower>
+	  </limit>
+	</axis>
+      </joint>
+    </xacro:macro>
+</robot>
