Commit message: wrapping up

File: urdf/quadrotor.urdf.xacro (robot description, xacro)
@@ -1,7 +1,35 @@
 <?xml version="1.0"?>
-<robot name="quadrotor" xmlns:xacro="http://wiki.ros.org/xacro" >
+<robot name="quadrotor_full" xmlns:xacro="http://wiki.ros.org/xacro" >
+    <xacro:property name="ID" value="$(arg id)" />
+    <xacro:property name="robot_name" value="quadrotor_$(arg id)" />
+    <xacro:property name="M_PI" value="3.1415926535897931" />
     <!-- Included URDF Files -->
     <xacro:include filename="$(find imav_2017)/urdf/quadrotor_base.urdf.xacro" />
-    <!-- Instantiate quadrotor_base_macro once (has no parameters atm) -->
-    <quadrotor_base_macro />
+    <!-- Base airframe -->
+    <quadrotor_base_macro/>
+    <xacro:include filename="$(find imav_2017)/urdf/sensors/quadrotor_sensors.urdf.xacro" />
+    <quadrotor_sensors robot_name="${robot_name}"/>
+    <xacro:include filename="$(find imav_2017)/urdf/quadrotor_simple_controller.urdf.xacro" />
+    <quadrotor_controller/>
+    <!-- Sonar height sensor -->
+    <xacro:include filename="$(find imav_2017)/urdf/sensors/sonar_sensor.urdf.xacro" />
+    <xacro:sonar_sensor name="sonar" parent="base_link" sim_name="${robot_name}" ros_topic="sonar_height" update_rate="10" min_range="0.01" max_range="3.0" field_of_view="${40*M_PI/180}" ray_count="3">
+      <origin xyz="-0.15 0.0 0.0" rpy="0 ${90*M_PI/180} 0"/>
+    </xacro:sonar_sensor>
+    <!-- Hokuyo UTM-30LX mounted upside down below the quadrotor body -->
+    <xacro:include filename="$(find imav_2017)/urdf/sensors/hokuyo_utm30lx.urdf.xacro" />
+    <xacro:hokuyo_utm30lx name="laser0" robot_name="${robot_name}" parent="base_link" ros_topic="scan" update_rate="40" ray_count="1081" min_angle="135" max_angle="-135">
+      <origin xyz="0.0 0.0 0.08" rpy="${M_PI} 0 0"/>
+    </xacro:hokuyo_utm30lx>
+    <!-- The following two cameras should be united to one! -->
+    <!-- Forward facing camera -->
+    <xacro:include filename="$(find imav_2017)/urdf/sensors/generic_camera.urdf.xacro" />
+    <xacro:generic_camera name="front" sim_name="${robot_name}" parent="base_link" update_rate="60" res_x="640" res_y="360" image_format="R8G8B8" hfov="${81*M_PI/180}">
+      <origin xyz="0.21 0.0 0.01" rpy="0 0 0"/>
+    </xacro:generic_camera>
+    <!-- Downward facing camera -->
+    <xacro:include filename="$(find imav_2017)/urdf/sensors/generic_camera.urdf.xacro" />
+    <xacro:generic_camera name="bottom" sim_name="${robot_name}" parent="base_link" update_rate="60" res_x="640" res_y="360" image_format="R8G8B8" hfov="${81*M_PI/180}">
+      <origin xyz="0.15 0.0 0.0" rpy="0 ${M_PI/2} 0"/>
+    </xacro:generic_camera>
 </robot>

File: urdf/quadrotor_base.urdf.xacro (robot description, xacro)
@@ -1,5 +1,7 @@
 <?xml version="1.0"?>
 <robot xmlns:xacro="http://wiki.ros.org/xacro" >
+<!--
   <xacro:include filename="$(find imav_2017)/plugins/urdf/quadrotor_plugins.urdf.xacro" />
+  -->
 <!--
   <xacro:property name="pi" value="3.1415926535897931" />
@@ -27,5 +29,7 @@
       </collision>
     </link>
+<!--
     <quadrotor_plugins/>
+    -->
   </xacro:macro>
 </robot>

File: urdf/quadrotor_simple_controller.urdf.xacro (robot description, xacro)
@@ -4,5 +4,8 @@
   <xacro:macro name="quadrotor_controller">
     <gazebo>
+      <!--
       <plugin name="quadrotor_simple_controller" filename="libquadrotor_simple_controller.so">
+      -->
+      <plugin name="quadrotor_simple_controller" filename="libgazebo_quadrotor_simple_controller.so">
         <alwaysOn>true</alwaysOn>
         <updateRate>0.0</updateRate>

File: urdf/sensors/generic_camera.urdf.xacro (robot description, xacro)
@@ -72,5 +72,5 @@
         </camera>
         <plugin name="${name}_camera_controller" filename="libgazebo_ros_camera.so">
-	  <cameraName>/${sim_name}/${name}</cameraName>
+	  <cameraName>/${robot_name}/${name}</cameraName>
           <alwaysOn>true</alwaysOn>
           <updateRate>${update_rate}</updateRate>

File: urdf/sensors/hokuyo_utm30lx.urdf.xacro (robot description, xacro)
@@ -1,6 +1,5 @@
 <?xml version="1.0"?>
 <robot xmlns:xacro="http://wiki.ros.org/xacro" >
-    <!--
-    <xacro:macro name="hokuyo_utm30lx" params="name parent *origin ros_topic update_rate ray_count min_angle max_angle">
+    <xacro:macro name="hokuyo_utm30lx" params="name parent robot_name *origin ros_topic update_rate ray_count min_angle max_angle">
       <joint name="${name}_joint" type="fixed">
 	<xacro:insert_block name="origin" />
@@ -29,44 +28,33 @@
       </link>
       <gazebo reference="${name}_frame">
-	<sensor:ray name="${name}">
-	  <rayCount>${ray_count}</rayCount>
-	  <rangeCount>${ray_count}</rangeCount>
-	  <laserCount>1</laserCount>
-	  <origin>0.0 0.0 0.0</origin>
-	  <displayRays>false</displayRays>
-	  <minAngle>${min_angle}</minAngle>
-	  <maxAngle>${max_angle}</maxAngle>
-	  <minRange>0.08</minRange>
-	  <maxRange>30.0</maxRange>
-	  <resRange>0.01</resRange>
-	  <updateRate>${update_rate}</updateRate>
-	  <controller:gazebo_ros_laser name="gazebo_ros_${name}_controller" plugin="libgazebo_ros_laser.so">
-	    <gaussianNoise>0.005</gaussianNoise>
-	    <alwaysOn>true</alwaysOn>
-	    <updateRate>${update_rate}</updateRate>
-	    <topicName>${ros_topic}</topicName>
-	    <frameName>${name}_frame</frameName>
-	    <interface:laser name="gazebo_ros_${name}_iface" />
-	  </controller:gazebo_ros_laser>
-	</sensor:ray>
+        <sensor type="ray" name="${name}">
+          <always_on>true</always_on>
+          <update_rate>${update_rate}</update_rate>
+          <pose>0 0 0 0 0 0</pose>
+          <visualize>false</visualize>
+          <ray>
+            <scan>
+              <horizontal>
+                <samples>${ray_count}</samples>
+                <resolution>1</resolution>
+                <min_angle>${min_angle * M_PI/180}</min_angle>
+                <max_angle>${max_angle * M_PI/180}</max_angle>
+              </horizontal>
+            </scan>
+            <range>
+              <min>0.08</min>
+              <max>30.0</max>
+              <resolution>0.01</resolution>
+            </range>
+          </ray>
+          <plugin name="gazebo_ros_${name}_controller" filename="libgazebo_ros_laser.so">
+            <gaussianNoise>0.005</gaussianNoise>
+            <alwaysOn>true</alwaysOn>
+            <updateRate>${update_rate}</updateRate>
+            <topicName>/${robot_name}/${ros_topic}</topicName>
+            <frameName>${name}_frame</frameName>
+          </plugin>
+        </sensor>
       </gazebo>
     </xacro:macro>
-    -->
-  <xacro:macro name="hokuyo" params="parent ros_topic update_rate ray_count min_angle max_angle">
-      <include>
-	<uri>model://hokuyo</uri>
-	<pose>0.2 0 0.2 0 0 0</pose>
-      </include>
-      <joint name="hokuyo_joint" type="revolute">
-	<child>hokuyo::link</child>
-	<parent>${parent}</parent>
-	<axis>
-	  <xyz>0 0 1</xyz>
-	  <limit>
-	    <upper>0</upper>
-	    <lower>0</lower>
-	  </limit>
-	</axis>
-      </joint>
-    </xacro:macro>
 </robot>

File: urdf/sensors/quadrotor_sensors.urdf.xacro (robot description, xacro)
@@ -4,5 +4,5 @@
         <frameId>ardrone_base_link</frameId>
 -->
-  <xacro:macro name="quadrotor_sensors">
+  <xacro:macro name="quadrotor_sensors" params="robot_name">
     <gazebo>
       <plugin name="quadrotor_imu_sim" filename="libhector_gazebo_ros_imu.so">
@@ -11,5 +11,5 @@
         <bodyName>base_link</bodyName>
         <frameId>ardrone_base_link</frameId>
-        <topicName>/ardrone/imu</topicName>
+        <topicName>/${robot_name}/imu</topicName>
         <rpyOffsets>0 0 0</rpyOffsets> <!-- deprecated -->
         <gaussianNoise>0</gaussianNoise>  <!-- deprecated -->
@@ -25,5 +25,5 @@
         <updateRate>10.0</updateRate>
         <bodyName>base_link</bodyName>
-        <topicName>pressure_height</topicName>
+        <topicName>/${robot_name}/pressure_height</topicName>
         <altimeterTopicName>altimeter</altimeterTopicName>
         <offset>0</offset>
@@ -35,5 +35,5 @@
         <updateRate>10.0</updateRate>
         <bodyName>base_link</bodyName>
-        <topicName>magnetic</topicName>
+        <topicName>/${robot_name}/magnetic</topicName>
         <offset>0 0 0</offset>
         <drift>0.0 0.0 0.0</drift>
@@ -44,6 +44,6 @@
         <updateRate>4.0</updateRate>
         <bodyName>base_link</bodyName>
-        <topicName>fix</topicName>
-        <velocityTopicName>fix_velocity</velocityTopicName>
+        <topicName>/${robot_name}/fix</topicName>
+        <velocityTopicName>/${robot_name}/fix_velocity</velocityTopicName>
         <drift>5.0 5.0 5.0</drift>
         <gaussianNoise>0.1 0.1 0.1</gaussianNoise>
@@ -55,5 +55,5 @@
         <updateRate>100.0</updateRate>
         <bodyName>base_link</bodyName>
-        <topicName>ground_truth/state</topicName>
+        <topicName>/${robot_name}/ground_truth/state</topicName>
         <gaussianNoise>0.0</gaussianNoise>
         <frameName>map</frameName>

File: urdf/sensors/sonar_sensor.urdf.xacro (robot description, xacro)
@@ -1,5 +1,5 @@
 <?xml version="1.0"?>
 <robot xmlns:xacro="http://wiki.ros.org/xacro" >
-  <xacro:macro name="sonar_sensor" params="name parent *origin ros_topic update_rate min_range max_range field_of_view ray_count">
+  <xacro:macro name="sonar_sensor" params="name parent *origin sim_name ros_topic update_rate min_range max_range field_of_view ray_count">
     <joint name="${name}_joint" type="fixed">
       <xacro:insert_block name="origin" />
@@ -51,5 +51,5 @@
         <plugin name="gazebo_ros_${name}_controller" filename="libhector_gazebo_ros_sonar.so">
           <gaussianNoise>0.000</gaussianNoise>
-          <topicName>${ros_topic}</topicName>
+          <topicName>/${sim_name}/${ros_topic}</topicName>
           <frameId>${name}_link</frameId>
         </plugin>

Commit message: cmd_vel and ps2cmd script changed

File: urdf/quadrotor.urdf.xacro (robot description, xacro)
@@ -11,5 +11,5 @@
     <quadrotor_sensors robot_name="${robot_name}"/>
     <xacro:include filename="$(find imav_2017)/urdf/quadrotor_simple_controller.urdf.xacro" />
-    <quadrotor_controller/>
+    <quadrotor_controller robot_name="${robot_name}"/>
     <!-- Sonar height sensor -->
     <xacro:include filename="$(find imav_2017)/urdf/sensors/sonar_sensor.urdf.xacro" />

File: urdf/quadrotor_simple_controller.urdf.xacro (robot description, xacro)
@@ -2,5 +2,5 @@
 <robot xmlns:xacro="http://wiki.ros.org/xacro" >
   <!-- Quadrotor Simple Controller Plugin -->
-  <xacro:macro name="quadrotor_controller">
+  <xacro:macro name="quadrotor_controller" params="robot_name">
     <gazebo>
       <plugin name="quadrotor_simple_controller" filename="libquadrotor_simple_controller.so">
@@ -10,5 +10,5 @@
         <!--<stateTopic>ground_truth/state</stateTopic>-->
         <!--<imuTopic>ardrone/imu</imuTopic>-->
-        <topicName>/cmd_vel</topicName>
+        <topicName>/${robot_name}/cmd_vel</topicName>
         <rollpitchProportionalGain>10.0</rollpitchProportionalGain>
         <rollpitchDifferentialGain>5.0</rollpitchDifferentialGain>

Commit message: xacro cleanup

File: urdf/quadrotor.urdf.xacro (robot description, xacro)
@@ -5,9 +5,11 @@
     <xacro:property name="M_PI" value="3.1415926535897931" />
     <!-- Included URDF Files -->
+    <!-- Base airframe -->
     <xacro:include filename="$(find imav_2017)/urdf/quadrotor_base.urdf.xacro" />
-    <!-- Base airframe -->
     <quadrotor_base_macro/>
+    <!-- IMU, Baro, Magnetic, GPS, Groundtruth sensors -->
     <xacro:include filename="$(find imav_2017)/urdf/sensors/quadrotor_sensors.urdf.xacro" />
     <quadrotor_sensors robot_name="${robot_name}"/>
+    <!-- 4D velocity control -->
     <xacro:include filename="$(find imav_2017)/urdf/quadrotor_simple_controller.urdf.xacro" />
     <quadrotor_controller robot_name="${robot_name}"/>
@@ -22,5 +24,4 @@
       <origin xyz="0.0 0.0 0.08" rpy="${M_PI} 0 0"/>
     </xacro:hokuyo_utm30lx>
-    <!-- The following two cameras should be united to one! -->
     <!-- Forward facing camera -->
     <xacro:include filename="$(find imav_2017)/urdf/sensors/generic_camera.urdf.xacro" />

File: urdf/quadrotor_base.urdf.xacro (robot description, xacro)
@@ -1,10 +1,4 @@
 <?xml version="1.0"?>
 <robot xmlns:xacro="http://wiki.ros.org/xacro" >
-<!--
-  <xacro:include filename="$(find imav_2017)/plugins/urdf/quadrotor_plugins.urdf.xacro" />
-  -->
-<!--
-  <xacro:property name="pi" value="3.1415926535897931" />
--->
   <!-- Main quadrotor link -->
   <xacro:macro name="quadrotor_base_macro">
@@ -29,7 +23,4 @@
       </collision>
     </link>
-<!--
-    <quadrotor_plugins/>
-    -->
   </xacro:macro>
 </robot>

File: urdf/sensors/generic_camera.urdf.xacro (robot description, xacro)
@@ -30,57 +30,57 @@
         </collision>
       </link>
-    <joint name="${name}_optical_joint" type="fixed">
-      <origin xyz="0 0 0" rpy="${-M_PI/2} 0.0 ${-M_PI/2}" />
-      <parent link="${name}_link" />
-      <child link="ardrone_base_${name}cam"/>
-    </joint>
-    <link name="ardrone_base_${name}cam">
-      <inertial>
-        <mass value="0.01" />
-        <origin xyz="0 0 0" />
-        <inertia ixx="0.001"  ixy="0.0"  ixz="0.0"
-                 iyy="0.001"  iyz="0.0"
-                 izz="0.001" />
-      </inertial>
-      <visual>
-        <origin xyz="0 0 0" rpy="0 0 0"/>
-        <geometry>
-          <box size="0.001 0.001 0.001" />
-        </geometry>
-      </visual>
-      <collision>
-        <origin xyz="0 0 0" rpy="0 0 0"/>
-        <geometry>
-          <box size="0.001 0.001 0.001" />
-        </geometry>
-      </collision>
-    </link>
-    <gazebo reference="${name}_link">
-      <sensor type="camera" name="${name}_camera_sensor">
-        <update_rate>${update_rate}</update_rate>
-        <camera name="head">
-          <horizontal_fov>${hfov}</horizontal_fov>
-          <image>
-            <width>${res_x}</width>
-            <height>${res_y}</height>
-            <format>${image_format}</format>
-          </image>
-          <clip>0.01
-	    <near>0.01</near>
-            <far>100</far>
-          </clip>
-        </camera>
-        <plugin name="${name}_camera_controller" filename="libgazebo_ros_camera.so">
-	  <cameraName>/${robot_name}/${name}</cameraName>
-          <alwaysOn>true</alwaysOn>
-          <updateRate>${update_rate}</updateRate>
-          <imageTopicName>/${sim_name}/${name}/image_raw</imageTopicName>
-          <cameraInfoTopicName>/${sim_name}/${name}/camera_info</cameraInfoTopicName>
-          <frameName>ardrone_base_${name}cam</frameName>
-        </plugin>
-      </sensor>
-      <!--<turnGravityOff>true</turnGravityOff>-->
-      <material>PR2/Blue</material>
-    </gazebo>
+      <joint name="${name}_optical_joint" type="fixed">
+	<origin xyz="0 0 0" rpy="${-M_PI/2} 0.0 ${-M_PI/2}" />
+	<parent link="${name}_link" />
+	<child link="ardrone_base_${name}cam"/>
+      </joint>
+      <link name="ardrone_base_${name}cam">
+	<inertial>
+	  <mass value="0.01" />
+	  <origin xyz="0 0 0" />
+	  <inertia ixx="0.001"  ixy="0.0"  ixz="0.0"
+		  iyy="0.001"  iyz="0.0"
+		  izz="0.001" />
+	</inertial>
+	<visual>
+	  <origin xyz="0 0 0" rpy="0 0 0"/>
+	  <geometry>
+	    <box size="0.001 0.001 0.001" />
+	  </geometry>
+	</visual>
+	<collision>
+	  <origin xyz="0 0 0" rpy="0 0 0"/>
+	  <geometry>
+	    <box size="0.001 0.001 0.001" />
+	  </geometry>
+	</collision>
+      </link>
+      <gazebo reference="${name}_link">
+	<sensor type="camera" name="${name}_camera_sensor">
+	  <update_rate>${update_rate}</update_rate>
+	  <camera name="head">
+	    <horizontal_fov>${hfov}</horizontal_fov>
+	    <image>
+	      <width>${res_x}</width>
+	      <height>${res_y}</height>
+	      <format>${image_format}</format>
+	    </image>
+	    <clip>0.01
+	      <near>0.01</near>
+	      <far>100</far>
+	    </clip>
+	  </camera>
+	  <plugin name="${name}_camera_controller" filename="libgazebo_ros_camera.so">
+	    <cameraName>/${robot_name}/${name}</cameraName>
+	    <alwaysOn>true</alwaysOn>
+	    <updateRate>${update_rate}</updateRate>
+	    <imageTopicName>/${sim_name}/${name}/image_raw</imageTopicName>
+	    <cameraInfoTopicName>/${sim_name}/${name}/camera_info</cameraInfoTopicName>
+	    <frameName>ardrone_base_${name}cam</frameName>
+	  </plugin>
+	</sensor>
+	<!--<turnGravityOff>true</turnGravityOff>-->
+	<material>PR2/Blue</material>
+      </gazebo>
     </xacro:macro>
-  </robot>
+</robot>

File: urdf/sensors/quadrotor_sensors.urdf.xacro (robot description, xacro)
@@ -1,7 +1,4 @@
 <?xml version="1.0"?>
 <robot xmlns:xacro="http://wiki.ros.org/xacro" >
-  <!-- Quadrotor Sensor Plugins
-        <frameId>ardrone_base_link</frameId>
--->
   <xacro:macro name="quadrotor_sensors" params="robot_name">
     <gazebo>

Commit message: Camera topic fixed

File: urdf/quadrotor.urdf.xacro (robot description, xacro)
@@ -26,10 +26,10 @@
     <!-- Forward facing camera -->
     <xacro:include filename="$(find imav_2017)/urdf/sensors/generic_camera.urdf.xacro" />
-    <xacro:generic_camera name="front" sim_name="${robot_name}" parent="base_link" update_rate="60" res_x="640" res_y="360" image_format="R8G8B8" hfov="${81*M_PI/180}">
+    <xacro:generic_camera name="front" robot_name="${robot_name}" parent="base_link" update_rate="60" res_x="640" res_y="360" image_format="R8G8B8" hfov="${81*M_PI/180}">
       <origin xyz="0.21 0.0 0.01" rpy="0 0 0"/>
     </xacro:generic_camera>
     <!-- Downward facing camera -->
     <xacro:include filename="$(find imav_2017)/urdf/sensors/generic_camera.urdf.xacro" />
-    <xacro:generic_camera name="bottom" sim_name="${robot_name}" parent="base_link" update_rate="60" res_x="640" res_y="360" image_format="R8G8B8" hfov="${81*M_PI/180}">
+    <xacro:generic_camera name="bottom" robot_name="${robot_name}" parent="base_link" update_rate="60" res_x="640" res_y="360" image_format="R8G8B8" hfov="${81*M_PI/180}">
       <origin xyz="0.15 0.0 0.0" rpy="0 ${M_PI/2} 0"/>
     </xacro:generic_camera>

File: urdf/sensors/generic_camera.urdf.xacro (robot description, xacro)
@@ -2,5 +2,5 @@
 <robot xmlns:xacro="http://wiki.ros.org/xacro">
     <xacro:property name="M_PI" value="3.1415926535897931" />
-    <xacro:macro name="generic_camera" params="name sim_name parent *origin update_rate res_x res_y image_format hfov">
+    <xacro:macro name="generic_camera" params="name parent robot_name *origin update_rate res_x res_y image_format hfov">
       <joint name="${name}_joint" type="fixed">
         <xacro:insert_block name="origin" />
@@ -73,9 +73,9 @@
 	  <plugin name="${name}_camera_controller" filename="libgazebo_ros_camera.so">
 	    <robotNamespace>${robot_name}</robotNamespace>
-	    <cameraName>/${robot_name}/${name}</cameraName>
+	    <cameraName>${name}</cameraName>
 	    <alwaysOn>true</alwaysOn>
 	    <updateRate>${update_rate}</updateRate>
-	    <imageTopicName>/${sim_name}/${name}/image_raw</imageTopicName>
-	    <cameraInfoTopicName>/${sim_name}/${name}/camera_info</cameraInfoTopicName>
+	    <imageTopicName>${name}/image_raw</imageTopicName>
+	    <cameraInfoTopicName>${name}/camera_info</cameraInfoTopicName>
 	    <frameName>ardrone_base_${name}cam</frameName>
 	  </plugin>
