Commit message: Tree collision fixed + launch handles xacro

File: worlds/xacro/macros.urdf.xacro (robot description, xacro)
@@ -310,4 +310,13 @@
 	    </geometry>
 	  </visual>
+	  <collision name="collision">
+	    <pose>0 0 0 1.5708 0 0</pose>
+	    <geometry>
+	      <mesh>
+		<uri>file://$(find imav_2017)/worlds/xacro/tree1.dae</uri>
+		<scale>0.01 0.01 0.01</scale>
+	      </mesh>
+	    </geometry>
+	  </collision>
 	</link>
       </model>

Commit message: Fix indentation

File: worlds/xacro/macros.urdf.xacro (robot description, xacro)
@@ -36,5 +36,5 @@
           </geometry>
           <material>
-	    <ambient>${color} 0.5</ambient>
+            <ambient>${color} 0.5</ambient>
           </material>
         </visual>
@@ -77,7 +77,7 @@
       <background>${backg}</background>
       <sky>
-	<clouds>
-	  <speed>12</speed>
-	</clouds>
+        <clouds>
+          <speed>12</speed>
+        </clouds>
       </sky>
       <shadows>1</shadows>
@@ -88,36 +88,36 @@
     <gui fullscreen='0'>
       <camera name='user_camera'>
-	<pose>1.49016 -3.72367 3.62379 -2.88294e-17 0.273797 1.4042</pose>
-	<view_controller>orbit</view_controller>
+        <pose>1.49016 -3.72367 3.62379 -2.88294e-17 0.273797 1.4042</pose>
+        <view_controller>orbit</view_controller>
       </camera>
     </gui>
   </xacro:macro>
   <xacro:macro name="wall_part" params="id w h l x y z">
-      <collision name="wall_p${id}_collision">
-	<pose>${x} ${y} ${z} 0 0 0</pose>
-	<geometry>
-	  <box>
-	    <size>${w} ${l} ${h}</size>
-	  </box>
-	</geometry>
-	<surface>
-	  <contact>
-	    <collide_bitmask>0x02</collide_bitmask>
-	  </contact>
-	</surface>
-      </collision>
-      <visual name="wall_p${id}_visual">
-	<pose>${x} ${y} ${z} 0 0 0</pose>
-	<geometry>
-	  <box>
-	    <size>${w} ${l} ${h}</size>
-	  </box>
-	</geometry>
-	<material>
-	  <script>
-	    <name>Gazebo/Wood</name>
-	  </script>
-	</material>
-      </visual>
+    <collision name="wall_p${id}_collision">
+      <pose>${x} ${y} ${z} 0 0 0</pose>
+      <geometry>
+        <box>
+          <size>${w} ${l} ${h}</size>
+        </box>
+      </geometry>
+      <surface>
+        <contact>
+          <collide_bitmask>0x02</collide_bitmask>
+        </contact>
+      </surface>
+    </collision>
+    <visual name="wall_p${id}_visual">
+      <pose>${x} ${y} ${z} 0 0 0</pose>
+      <geometry>
+        <box>
+          <size>${w} ${l} ${h}</size>
+        </box>
+      </geometry>
+      <material>
+        <script>
+          <name>Gazebo/Wood</name>
+        </script>
+      </material>
+    </visual>
   </xacro:macro>
   <xacro:macro name="wall_brand" params="w h l x y z">
@@ -126,32 +126,32 @@
       <pose>${x} ${y} ${z} 0 0 0</pose>
       <link name="wall_link">
-	<inertial>
-	  <mass>10000</mass>
-	</inertial>
-	<collision name="wall_brand_collision">
-	  <geometry>
-	    <box>
-	      <size>${w} ${l} ${h}</size>
-	    </box>
-	  </geometry>
-	  <surface>
-	    <contact>
-	      <collide_bitmask>0x02</collide_bitmask>
-	    </contact>
-	  </surface>
-	</collision>
-	<visual name="wall_brand_visual">
-	  <geometry>
-	    <box>
-	      <size>${w} ${l} ${h}</size>
-	    </box>
-	  </geometry>
-	  <material>
-	    <script>
-	      <uri>file://$(find imav_2017)/worlds/xacro/custom.material</uri>
-	      <name>MathWorks_branding</name>
-	    </script>
-	  </material>
-	</visual>
+        <inertial>
+          <mass>10000</mass>
+        </inertial>
+        <collision name="wall_brand_collision">
+          <geometry>
+            <box>
+              <size>${w} ${l} ${h}</size>
+            </box>
+          </geometry>
+          <surface>
+            <contact>
+              <collide_bitmask>0x02</collide_bitmask>
+            </contact>
+          </surface>
+        </collision>
+        <visual name="wall_brand_visual">
+          <geometry>
+            <box>
+              <size>${w} ${l} ${h}</size>
+            </box>
+          </geometry>
+          <material>
+            <script>
+              <uri>file://$(find imav_2017)/worlds/xacro/custom.material</uri>
+              <name>MathWorks_branding</name>
+            </script>
+          </material>
+        </visual>
       </link>
     </model>
@@ -162,21 +162,21 @@
       <pose>${offset} 0 ${height/2} 0 0 0</pose>
       <link name="wall_link">
-	<inertial>
-	  <mass>10000</mass>
-	</inertial>
-	<xacro:wall_part id="1"  w="0.2" h="${height}" 		l="${(5-w_b)/2}" 	x="0" y="${ (w_b/2+(5-w_b)/4)}"	z="0"/>
-	<xacro:wall_part id="2"  w="0.2" h="${height}" 		l="2" 			x="0" y="${ (2.5+w_s+1)}" 	z="0"/>
-	<xacro:wall_part id="3"  w="0.2" h="${height}" 		l="${(5-w_b)/2}" 	x="0" y="${-(w_b/2+(5-w_b)/4)}"	z="0"/>
-	<xacro:wall_part id="4"  w="0.2" h="${height}" 		l="2" 			x="0" y="${-(2.5+w_s+1)}" 	z="0"/>
-	<xacro:wall_part id="5"  w="0.2" h="${(height-w_b)/2}"	l="${w_b}"   		x="0" y="0" 			z="${-((height-w_b)/4+w_b/2)}"/>
-	<xacro:wall_part id="6"  w="0.2" h="${(height-w_s)/2}"	l="${w_s}" 		x="0" y="${ (2.5+w_s/2)}"	z="${-((height-w_s)/4+w_s/2)}"/>
-	<xacro:wall_part id="7"  w="0.2" h="${(height-w_s)/2}"	l="${w_s}" 		x="0" y="${-(2.5+w_s/2)}"	z="${-((height-w_s)/4+w_s/2)}"/>
-	<xacro:wall_part id="8"  w="0.2" h="${(height-w_b)/2}"	l="${w_b}"   		x="0" y="0" 			z="${ ((height-w_b)/4+w_b/2)}"/>
-	<xacro:wall_part id="9"  w="0.2" h="${(height-w_s)/2}"	l="${w_s}" 		x="0" y="${ (2.5+w_s/2)}"	z="${ ((height-w_s)/4+w_s/2)}"/>
-	<xacro:wall_part id="10" w="0.2" h="${(height-w_s)/2}"	l="${w_s}" 		x="0" y="${-(2.5+w_s/2)}"	z="${ ((height-w_s)/4+w_s/2)}"/>
-	<xacro:wall_part id="11" w="${l_p}" h="0.2"		l="${w_s+0.3998}" 		x="0" y="${ (2.5+w_s/2)}"		z="${-(w_s/2+0.099)}"/>
-	<xacro:wall_part id="12" w="${l_p}" h="0.2"		l="${w_s+0.3998}" 		x="0" y="${ (2.5+w_s/2)}"		z="${ (w_s/2+0.099)}"/>
-	<xacro:wall_part id="13" w="${l_p}" h="${w_s-0.001}"	l="0.2" 		x="0" y="${ (2.5+w_s/2)-(w_s/2)-0.099}"	z="0.0"/>
-	<xacro:wall_part id="14" w="${l_p}" h="${w_s-0.001}"	l="0.2" 		x="0" y="${ (2.5+w_s/2)+(w_s/2)+0.099}"	z="0.0"/>
+        <inertial>
+          <mass>10000</mass>
+        </inertial>
+        <xacro:wall_part id="1"  w="0.2" h="${height}" 		l="${(5-w_b)/2}" 	x="0" y="${ (w_b/2+(5-w_b)/4)}"	z="0"/>
+        <xacro:wall_part id="2"  w="0.2" h="${height}" 		l="2" 			x="0" y="${ (2.5+w_s+1)}" 	z="0"/>
+        <xacro:wall_part id="3"  w="0.2" h="${height}" 		l="${(5-w_b)/2}" 	x="0" y="${-(w_b/2+(5-w_b)/4)}"	z="0"/>
+        <xacro:wall_part id="4"  w="0.2" h="${height}" 		l="2" 			x="0" y="${-(2.5+w_s+1)}" 	z="0"/>
+        <xacro:wall_part id="5"  w="0.2" h="${(height-w_b)/2}"	l="${w_b}"   		x="0" y="0" 			z="${-((height-w_b)/4+w_b/2)}"/>
+        <xacro:wall_part id="6"  w="0.2" h="${(height-w_s)/2}"	l="${w_s}" 		x="0" y="${ (2.5+w_s/2)}"	z="${-((height-w_s)/4+w_s/2)}"/>
+        <xacro:wall_part id="7"  w="0.2" h="${(height-w_s)/2}"	l="${w_s}" 		x="0" y="${-(2.5+w_s/2)}"	z="${-((height-w_s)/4+w_s/2)}"/>
+        <xacro:wall_part id="8"  w="0.2" h="${(height-w_b)/2}"	l="${w_b}"   		x="0" y="0" 			z="${ ((height-w_b)/4+w_b/2)}"/>
+        <xacro:wall_part id="9"  w="0.2" h="${(height-w_s)/2}"	l="${w_s}" 		x="0" y="${ (2.5+w_s/2)}"	z="${ ((height-w_s)/4+w_s/2)}"/>
+        <xacro:wall_part id="10" w="0.2" h="${(height-w_s)/2}"	l="${w_s}" 		x="0" y="${-(2.5+w_s/2)}"	z="${ ((height-w_s)/4+w_s/2)}"/>
+        <xacro:wall_part id="11" w="${l_p}" h="0.2"		l="${w_s+0.3998}" 		x="0" y="${ (2.5+w_s/2)}"		z="${-(w_s/2+0.099)}"/>
+        <xacro:wall_part id="12" w="${l_p}" h="0.2"		l="${w_s+0.3998}" 		x="0" y="${ (2.5+w_s/2)}"		z="${ (w_s/2+0.099)}"/>
+        <xacro:wall_part id="13" w="${l_p}" h="${w_s-0.001}"	l="0.2" 		x="0" y="${ (2.5+w_s/2)-(w_s/2)-0.099}"	z="0.0"/>
+        <xacro:wall_part id="14" w="${l_p}" h="${w_s-0.001}"	l="0.2" 		x="0" y="${ (2.5+w_s/2)+(w_s/2)+0.099}"	z="0.0"/>
       </link>
     </model>
@@ -220,48 +220,48 @@
       <pose>${x} ${y} ${z} 0 0 0</pose>
       <collision name='collision'>
-	<geometry>
-	  <box>
-	    <size>${size}</size>
-	  </box>
-	</geometry>
+        <geometry>
+          <box>
+            <size>${size}</size>
+          </box>
+        </geometry>
       </collision>
       <visual name='visual'>
-	<geometry>
-	  <box>
-	    <size>${size}</size>
-	  </box>
-	</geometry>
+        <geometry>
+          <box>
+            <size>${size}</size>
+          </box>
+        </geometry>
       </visual>
     </link>
   </xacro:macro>
   <xacro:macro name="pole" params="id h r x y z">
-      <collision name="pole_p${id}_collision">
-	<pose>${x} ${y} ${z} 0 0 0</pose>
-	<geometry>
-	  <cylinder>
-	    <radius>${r}</radius>
-	    <length>${h}</length>
-	  </cylinder>
-	</geometry>
-	<surface>
-	  <contact>
-	    <collide_bitmask>0x02</collide_bitmask>
-	  </contact>
-	</surface>
-      </collision>
-      <visual name="pole_p${id}_visual">
-	<pose>${x} ${y} ${z} 0 0 0</pose>
-	<geometry>
-	  <cylinder>
-	    <radius>${r}</radius>
-	    <length>${h}</length>
-	  </cylinder>
-	</geometry>
-	<material>
-	  <script>
-	    <name>Gazebo/Bricks</name>
-	  </script>
-	</material>
-      </visual>
+    <collision name="pole_p${id}_collision">
+      <pose>${x} ${y} ${z} 0 0 0</pose>
+      <geometry>
+        <cylinder>
+          <radius>${r}</radius>
+          <length>${h}</length>
+        </cylinder>
+      </geometry>
+      <surface>
+        <contact>
+          <collide_bitmask>0x02</collide_bitmask>
+        </contact>
+      </surface>
+    </collision>
+    <visual name="pole_p${id}_visual">
+      <pose>${x} ${y} ${z} 0 0 0</pose>
+      <geometry>
+        <cylinder>
+          <radius>${r}</radius>
+          <length>${h}</length>
+        </cylinder>
+      </geometry>
+      <material>
+        <script>
+          <name>Gazebo/Bricks</name>
+        </script>
+      </material>
+    </visual>
   </xacro:macro>
   <xacro:macro name="pole2" params="h r">
@@ -269,28 +269,28 @@
     <link name="pole_link">
       <collision name="pole_collision">
-	<geometry>
-	  <cylinder>
-	    <radius>${r}</radius>
-	    <length>${h}</length>
-	  </cylinder>
-	</geometry>
-	<surface>
-	  <contact>
-	    <collide_bitmask>0x02</collide_bitmask>
-	  </contact>
-	</surface>
+        <geometry>
+          <cylinder>
+            <radius>${r}</radius>
+            <length>${h}</length>
+          </cylinder>
+        </geometry>
+        <surface>
+          <contact>
+            <collide_bitmask>0x02</collide_bitmask>
+          </contact>
+        </surface>
       </collision>
       <visual name="pole_visual">
-	<geometry>
-	  <cylinder>
-	    <radius>${r}</radius>
-	    <length>${h}</length>
-	  </cylinder>
-	</geometry>
-	<material>
-	  <script>
-	    <name>Gazebo/Bricks</name>
-	  </script>
-	</material>
+        <geometry>
+          <cylinder>
+            <radius>${r}</radius>
+            <length>${h}</length>
+          </cylinder>
+        </geometry>
+        <material>
+          <script>
+            <name>Gazebo/Bricks</name>
+          </script>
+        </material>
       </visual>
     </link>
@@ -299,5 +299,5 @@
     <population name="pole_population">
       <model name="pole">
-	<xacro:pole2 h="${h}" r="${r}"/>
+        <xacro:pole2 h="${h}" r="${r}"/>
       </model>
       <pose>${x} ${y} ${h/2} 0 0 0</pose>
@@ -316,15 +316,15 @@
       <pose>${x} ${y} ${h/2} 0 0 0</pose>
       <link name="poles_link">
-	<inertial>
-	  <mass>10000</mass>
-	</inertial>
-	<xacro:pole id="1" h="${h}" r="${r}" x="0" 		y="${w/4}" z="0"/>
-	<xacro:pole id="2" h="${h}" r="${r}" x="${ 2*l/6}" 	y="${w/4}" z="0"/>
-	<xacro:pole id="3" h="${h}" r="${r}" x="${-2*l/6}" 	y="${w/4}" z="0"/>
-	<xacro:pole id="4" h="${h}" r="${r}" x="${ l/6}" 	y="0" z="0"/>
-	<xacro:pole id="5" h="${h}" r="${r}" x="${-l/6}" 	y="0" z="0"/>
-	<xacro:pole id="6" h="${h}" r="${r}" x="0"	 	y="${-w/4}" z="0"/>
-	<xacro:pole id="7" h="${h}" r="${r}" x="${ 2*l/6}" 	y="${-w/4}" z="0"/>
-	<xacro:pole id="8" h="${h}" r="${r}" x="${-2*l/6}" 	y="${-w/4}" z="0"/>
+        <inertial>
+          <mass>10000</mass>
+        </inertial>
+        <xacro:pole id="1" h="${h}" r="${r}" x="0" 		y="${w/4}" z="0"/>
+        <xacro:pole id="2" h="${h}" r="${r}" x="${ 2*l/6}" 	y="${w/4}" z="0"/>
+        <xacro:pole id="3" h="${h}" r="${r}" x="${-2*l/6}" 	y="${w/4}" z="0"/>
+        <xacro:pole id="4" h="${h}" r="${r}" x="${ l/6}" 	y="0" z="0"/>
+        <xacro:pole id="5" h="${h}" r="${r}" x="${-l/6}" 	y="0" z="0"/>
+        <xacro:pole id="6" h="${h}" r="${r}" x="0"	 	y="${-w/4}" z="0"/>
+        <xacro:pole id="7" h="${h}" r="${r}" x="${ 2*l/6}" 	y="${-w/4}" z="0"/>
+        <xacro:pole id="8" h="${h}" r="${r}" x="${-2*l/6}" 	y="${-w/4}" z="0"/>
       </link>
     </model>
@@ -333,25 +333,25 @@
     <population name="tree_population">
       <model name="tree">
-	<static>true</static>
-	<link name="body">
-	  <visual name="visual">
-	    <pose>0 0 0 1.5708 0 0</pose>
-	    <geometry>
-	      <mesh>
-		<uri>file://$(find imav_2017)/worlds/xacro/tree1.dae</uri>
-		<scale>0.01 0.01 0.01</scale>
-	      </mesh>
-	    </geometry>
-	  </visual>
-	  <collision name="collision">
-	    <pose>0 0 0 1.5708 0 0</pose>
-	    <geometry>
-	      <mesh>
-		<uri>file://$(find imav_2017)/worlds/xacro/tree1.dae</uri>
-		<scale>0.01 0.01 0.01</scale>
-	      </mesh>
-	    </geometry>
-	  </collision>
-	</link>
+        <static>true</static>
+        <link name="body">
+          <visual name="visual">
+            <pose>0 0 0 1.5708 0 0</pose>
+            <geometry>
+              <mesh>
+                <uri>file://$(find imav_2017)/worlds/xacro/tree1.dae</uri>
+                <scale>0.01 0.01 0.01</scale>
+              </mesh>
+            </geometry>
+          </visual>
+          <collision name="collision">
+            <pose>0 0 0 1.5708 0 0</pose>
+            <geometry>
+              <mesh>
+                <uri>file://$(find imav_2017)/worlds/xacro/tree1.dae</uri>
+                <scale>0.01 0.01 0.01</scale>
+              </mesh>
+            </geometry>
+          </collision>
+        </link>
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