Commit message: Helipad fixed

File: worlds/xacro/imav_indoor.world.xacro (robot description, xacro)
@@ -3,7 +3,7 @@
   <world name="imav_world" xmlns:xacro="http://www.ros.org/wiki/xacro">
     <xacro:property name="width" value="13" />
-    <xacro:property name="length1" value="30" />
-    <xacro:property name="length2" value="30" />
-    <xacro:property name="length3" value="30" />
+    <xacro:property name="length1" value="10" />
+    <xacro:property name="length2" value="10" />
+    <xacro:property name="length3" value="13" />
     <xacro:include filename="$(find imav_2017)/worlds/xacro/macros.urdf.xacro" />
     <xacro:light_source/>
@@ -19,11 +19,11 @@
     <xacro:wall_obstacle w_s="0.5" w_b="1" w_t="0.5" offset="${length1/4}" width="${width}" height="3"/>
     <xacro:wall_brand w="${length1+length2+length3}" h="${3*3}"	l="0.2" x="${length1/2+length2/2}" y="${width*2}"	z="${3*3/2}"/>
-    <xacro:poles2 h="3" r="0.25" w="${width}" l="${length2}" x="${length1/2+length2/2}" y="0" num="50"/>
+    <xacro:poles2 h="3" r="0.25" w="${width*3/4}" l="${length2}" x="${length1/2+length2/2}" y="${width/8}" num="20"/>
     <!--
     <xacro:trees w="${width}" l="${length2/2}" x="${length1/2+3*length2/4}" y="0"/>
     <xacro:bushes w="${width}" l="${length2/2}" x="${length1/2+3*length2/4}" y="0"/>
     -->
-    <xacro:helipad_static size="0.5 0.5 0.01" x="1"  y="1"  z="0.1"/>
-    <xacro:helipad_mobile size="0.5 0.5 0.01" x="-1" y="-1" z="0.1" r="1" v="1"/>
+    <xacro:helipad_static size="1 1 0.01" x="-2.5"  y="2.5"  z="0.1"/>
+    <xacro:helipad_mobile size="1 1 0.01" x="-2.5" y="-2.5" z="0.1" r="1" v="1"/>
   </world>
 </sdf>

File: worlds/xacro/macros.urdf.xacro (robot description, xacro)
@@ -178,4 +178,23 @@
     </model>
   </xacro:macro>
+  <xacro:macro name="box_" params="name x y z size">
+    <link name='${name}'>
+      <pose>${x} ${y} ${z} 0 0 0</pose>
+      <collision name='collision'>
+	<geometry>
+	  <box>
+	    <size>${size}</size>
+	  </box>
+	</geometry>
+      </collision>
+      <visual name='visual'>
+	<geometry>
+	  <box>
+	    <size>${size}</size>
+	  </box>
+	</geometry>
+      </visual>
+    </link>
+  </xacro:macro>
   <xacro:macro name="pole" params="id h r x y z">
       <collision name="pole_p${id}_collision">
@@ -250,5 +269,5 @@
       <model_count>${num}</model_count>
       <distribution>
-        <type>random</type>
+        <type>uniform</type>
       </distribution>
     </population>
@@ -345,5 +364,5 @@
     <model name="helipad_static">
       <static>true</static>
-      <xacro:helipad size="${size}" x="${x+1}" y="${y}" z="${z}"/>
+      <xacro:helipad size="${size}" x="${x}" y="${y}" z="${z}"/>
     </model>
   </xacro:macro>
@@ -351,8 +370,15 @@
     <model name="helipad_mobile">
       <pose>${x} ${y} ${z} 0 0 0</pose>
+      <self_collide>false</self_collide>
+      <joint name="helipad_fix0" type="fixed">
+	  <pose>0 0 0 0 0 0</pose>
+	  <parent>world</parent>
+	  <child>base</child>
+      </joint>
+      <xacro:box_ name='base' size="0.2 0.2 0.2" x="0" y="0" z="0"/>
       <joint name="helipad_joint" type="revolute">
-	<pose>${x} ${y} ${z} 0 0 0</pose>
-	<parent>world</parent>
-	<child>helipad_link</child>
+	<pose>-${r/2} 0 0 0 0 0</pose>
+	<parent>base</parent>
+	<child>arm</child>
 	<axis>
 	  <xyz>0 0 1</xyz>
@@ -365,5 +391,11 @@
 	</physics>
       </joint>
-      <xacro:helipad size="${size}" x="${1}" y="0" z="0"/>
+      <xacro:box_ name='arm' size="${r} 0.2 0.01" x="${r/2}" y="0" z="0.095"/>
+      <joint name="helipad_fix1" type="fixed">
+	<pose>0 0 0 0 0 0</pose>
+	<parent>arm</parent>
+	<child>helipad_link</child>
+      </joint>
+      <xacro:helipad size="${size}" x="${r}" y="0" z="0.1"/>
     </model>
   </xacro:macro>

Commit message: Wall fixed

File: worlds/xacro/imav_indoor.world.xacro (robot description, xacro)
@@ -17,5 +17,5 @@
     <xacro:zone name="obstacle" 	offset="${length1/2+length2/2}" 		width="${width}" length="${length2}" color="${188/255} ${53/255}  ${53/255}"/>
     <xacro:zone name="target" 		offset="${length1/2+length2+length3/2}" 	width="${width}" length="${length3}" color="${78/255}  ${83/255}  ${199/255}"/>
-    <xacro:wall_obstacle w_s="0.5" w_b="1" w_t="0.5" offset="${length1/4}" width="${width}" height="3"/>
+    <xacro:wall_obstacle w_s="1.0" w_b="1.5" w_t="1.0" l_p="2.0" offset="${length1/4}" width="${width}" height="3"/>
     <xacro:wall_brand w="${length1+length2+length3}" h="${3*3}"	l="0.2" x="${length1/2+length2/2}" y="${width*2}"	z="${3*3/2}"/>
     <xacro:poles2 h="3" r="0.25" w="${width*3/4}" l="${length2}" x="${length1/2+length2/2}" y="${width/8}" num="20"/>

File: worlds/xacro/macros.urdf.xacro (robot description, xacro)
@@ -157,5 +157,5 @@
     </model>
   </xacro:macro>
-  <xacro:macro name="wall_obstacle" params="w_s w_b w_t offset width height">
+  <xacro:macro name="wall_obstacle" params="w_s w_b w_t l_p offset width height">
     <model name="wall">
       <static>1</static>
@@ -165,14 +165,18 @@
 	  <mass>10000</mass>
 	</inertial>
-	<xacro:wall_part id="1"  w="0.2" h="${height}" l="2" x="0" y="${w_b/2+1}" z="0"/>
-	<xacro:wall_part id="2"  w="0.2" h="${height}" l="2" x="0" y="${w_b/2+2+1.5}" z="0"/>
-	<xacro:wall_part id="3"  w="0.2" h="${height}" l="2" x="0" y="${-(w_b/2+1)}" z="0"/>
-	<xacro:wall_part id="4"  w="0.2" h="${height}" l="2" x="0" y="${-(w_b/2+2+1.5)}" z="0"/>
-	<xacro:wall_part id="5"  w="0.2" h="1"	l="1"   x="0" y="0" 		z="-1.00"/>
-	<xacro:wall_part id="6"  w="0.2" h="1.5"	l="0.5" x="0" y="${0.75+2}"	z="-0.75"/>
-	<xacro:wall_part id="7"  w="0.2" h="1.5"	l="0.5" x="0" y="${-(0.75+2)}"	z="-0.75"/>
-	<xacro:wall_part id="8"  w="0.2" h="1"	l="1"   x="0" y="0" 		z="1.00"/>
-	<xacro:wall_part id="9"  w="0.2" h="1"	l="0.5" x="0" y="${0.75+2}"	z="1"/>
-	<xacro:wall_part id="10" w="0.2" h="1"	l="0.5" x="0" y="${-(0.75+2)}"	z="1"/>
+	<xacro:wall_part id="1"  w="0.2" h="${height}" 		l="${(5-w_b)/2}" 	x="0" y="${ (w_b/2+(5-w_b)/4)}"	z="0"/>
+	<xacro:wall_part id="2"  w="0.2" h="${height}" 		l="2" 			x="0" y="${ (2.5+w_s+1)}" 	z="0"/>
+	<xacro:wall_part id="3"  w="0.2" h="${height}" 		l="${(5-w_b)/2}" 	x="0" y="${-(w_b/2+(5-w_b)/4)}"	z="0"/>
+	<xacro:wall_part id="4"  w="0.2" h="${height}" 		l="2" 			x="0" y="${-(2.5+w_s+1)}" 	z="0"/>
+	<xacro:wall_part id="5"  w="0.2" h="${(height-w_b)/2}"	l="${w_b}"   		x="0" y="0" 			z="${-((height-w_b)/4+w_b/2)}"/>
+	<xacro:wall_part id="6"  w="0.2" h="${(height-w_s)/2}"	l="${w_s}" 		x="0" y="${ (2.5+w_s/2)}"	z="${-((height-w_s)/4+w_s/2)}"/>
+	<xacro:wall_part id="7"  w="0.2" h="${(height-w_s)/2}"	l="${w_s}" 		x="0" y="${-(2.5+w_s/2)}"	z="${-((height-w_s)/4+w_s/2)}"/>
+	<xacro:wall_part id="8"  w="0.2" h="${(height-w_b)/2}"	l="${w_b}"   		x="0" y="0" 			z="${ ((height-w_b)/4+w_b/2)}"/>
+	<xacro:wall_part id="9"  w="0.2" h="${(height-w_s)/2}"	l="${w_s}" 		x="0" y="${ (2.5+w_s/2)}"	z="${ ((height-w_s)/4+w_s/2)}"/>
+	<xacro:wall_part id="10" w="0.2" h="${(height-w_s)/2}"	l="${w_s}" 		x="0" y="${-(2.5+w_s/2)}"	z="${ ((height-w_s)/4+w_s/2)}"/>
+	<xacro:wall_part id="11" w="${l_p}" h="0.2"		l="${w_s+0.3998}" 		x="0" y="${ (2.5+w_s/2)}"		z="${-(w_s/2+0.099)}"/>
+	<xacro:wall_part id="12" w="${l_p}" h="0.2"		l="${w_s+0.3998}" 		x="0" y="${ (2.5+w_s/2)}"		z="${ (w_s/2+0.099)}"/>
+	<xacro:wall_part id="13" w="${l_p}" h="${w_s-0.001}"	l="0.2" 		x="0" y="${ (2.5+w_s/2)-(w_s/2)-0.099}"	z="0.0"/>
+	<xacro:wall_part id="14" w="${l_p}" h="${w_s-0.001}"	l="0.2" 		x="0" y="${ (2.5+w_s/2)+(w_s/2)+0.099}"	z="0.0"/>
       </link>
     </model>

Commit message: Poles, trees fixed

File: worlds/xacro/imav_indoor.world.xacro (robot description, xacro)
@@ -19,5 +19,6 @@
     <xacro:wall_obstacle w_s="1.0" w_b="1.5" w_t="1.0" l_p="2.0" offset="${length1/4}" width="${width}" height="3"/>
     <xacro:wall_brand w="${length1+length2+length3}" h="${3*3}"	l="0.2" x="${length1/2+length2/2}" y="${width*2}"	z="${3*3/2}"/>
-    <xacro:poles2 h="3" r="0.25" w="${width*3/4}" l="${length2}" x="${length1/2+length2/2}" y="${width/8}" num="20"/>
+    <xacro:poles2 h="3" r="0.25" 	w="${width*3/4}" l="${length2/2}" x="${length1/2+length2/4}"   y="${width/8}" num="10"/>
+    <xacro:trees  			w="${width*3/4}" l="${length2/2}" x="${length1/2+3*length2/4}" y="${width/8}" num="10"/>
     <!--
     <xacro:trees w="${width}" l="${length2/2}" x="${length1/2+3*length2/4}" y="0"/>

File: worlds/xacro/macros.urdf.xacro (robot description, xacro)
@@ -273,5 +273,5 @@
       <model_count>${num}</model_count>
       <distribution>
-        <type>uniform</type>
+        <type>random</type>
       </distribution>
     </population>
@@ -296,19 +296,27 @@
     </model>
   </xacro:macro>
-  <xacro:macro name="trees" params="w l x y">
-    <population name="pole_population">
-      <model name="pole">
-	<include>
-          <static>true</static>
-          <uri>model://meshes/tree.dae</uri>
-        </include>
+  <xacro:macro name="trees" params="w l x y num">
+    <population name="tree_population">
+      <model name="tree">
+	<static>true</static>
+	<link name="body">
+	  <visual name="visual">
+	    <pose>0 0 0 1.5708 0 0</pose>
+	    <geometry>
+	      <mesh>
+		<uri>file://$(find imav_2017)/worlds/xacro/tree1.dae</uri>
+		<scale>0.01 0.01 0.01</scale>
+	      </mesh>
+	    </geometry>
+	  </visual>
+	</link>
       </model>
-      <pose>${x} ${y} 0 0 0</pose>
+      <pose>${x} ${y} 0 0 0 0</pose>
       <box>
         <size>${l} ${w} 0.1</size>
       </box>
-      <model_count>10</model_count>
+      <model_count>${num}</model_count>
       <distribution>
-        <type>uniform</type>
+        <type>random</type>
       </distribution>
     </population>

Commit message: QR, X added

File: worlds/xacro/imav_indoor.world.xacro (robot description, xacro)
@@ -14,7 +14,7 @@
     <xacro:scn amb="0.4 0.4 0.4 1" backg="${53/255} ${147/255} ${37/255} 1"/>
     -->
-    <xacro:zone name="takoff_landing" 	offset="0"	 				width="${width}" length="${length1}" color="${22/255}  ${176/255} ${37/255}"/>
-    <xacro:zone name="obstacle" 	offset="${length1/2+length2/2}" 		width="${width}" length="${length2}" color="${188/255} ${53/255}  ${53/255}"/>
-    <xacro:zone name="target" 		offset="${length1/2+length2+length3/2}" 	width="${width}" length="${length3}" color="${78/255}  ${83/255}  ${199/255}"/>
+    <xacro:zone name="takoff_landing" 	x="0"	 				y = "0.0" width="${width}" length="${length1}" color="${22/255}  ${176/255} ${37/255}"/>
+    <xacro:zone name="obstacle" 	x="${length1/2+length2/2}" 		y = "0.0" width="${width}" length="${length2}" color="${188/255} ${53/255}  ${53/255}"/>
+    <xacro:zone name="target" 		x="${length1/2+length2+length3/2}" 	y = "0.0" width="${width}" length="${length3}" color="${78/255}  ${83/255}  ${199/255}"/>
     <xacro:wall_obstacle w_s="1.0" w_b="1.5" w_t="1.0" l_p="2.0" offset="${length1/4}" width="${width}" height="3"/>
     <xacro:wall_brand w="${length1+length2+length3}" h="${3*3}"	l="0.2" x="${length1/2+length2/2}" y="${width*2}"	z="${3*3/2}"/>
@@ -27,4 +27,9 @@
     <xacro:helipad_static size="1 1 0.01" x="-2.5"  y="2.5"  z="0.1"/>
     <xacro:helipad_mobile size="1 1 0.01" x="-2.5" y="-2.5" z="0.1" r="1" v="1"/>
+    <xacro:QR1 size="0.5 0.5 0.01" x="${length1/2+length2+length3/2}" 	y="${width/4}"  z="0.1"/>
+    <xacro:X1 size="2 2 0.01" x="${length1/2+length2+length3/2}" 	y="${-width/4}"  z="0.1"/>
+    <!--
+    <xacro:zone name="drop" 	x="${length1/2+length2+length3/2}" 	y="${-width/4}" width="2" length="2" color="${255/255}  ${0/255}  ${199/255}"/>
+    -->
   </world>
 </sdf>

File: worlds/xacro/macros.urdf.xacro (robot description, xacro)
@@ -1,8 +1,8 @@
 <?xml version="1.0"?>
 <my_macros xmlns:xacro="http://www.ros.org/wiki/xacro">
-  <xacro:macro name="zone" params="name offset width length color">
+  <xacro:macro name="zone" params="name width length color x y">
     <model name="${name}_zone">
       <static>1</static>
-      <pose>${offset} 0 0 0 0 0</pose>
+      <pose>${x} ${y} 0 0 0 0</pose>
       <link name='link'>
         <collision name='collision'>
@@ -412,3 +412,75 @@
     </model>
   </xacro:macro>
+  <xacro:macro name="QR1" params="size x y z">
+    <model name="QR">
+      <static>true</static>
+      <link name="QR1_link">
+	<pose>${x} ${y} ${z} 0 0 0</pose>
+	<inertial>
+	  <mass>10</mass>
+	</inertial>
+	<collision name="qr_collision">
+	  <geometry>
+	    <box>
+	      <size>${size}</size>
+	    </box>
+	  </geometry>
+	  <surface>
+	    <contact>
+	      <collide_bitmask>0x02</collide_bitmask>
+	    </contact>
+	  </surface>
+	</collision>
+	<visual name="qr_visual">
+	  <geometry>
+	    <box>
+	      <size>${size}</size>
+	    </box>
+	  </geometry>
+	  <material>
+	    <script>
+	      <uri>file://$(find imav_2017)/worlds/xacro/custom.material</uri>
+	      <name>QR1</name>
+	    </script>
+	  </material>
+	</visual>
+      </link>
+    </model>
+  </xacro:macro>
+  <xacro:macro name="X1" params="size x y z">
+    <model name="X">
+      <static>true</static>
+      <link name="X_link">
+	<pose>${x} ${y} ${z} 0 0 0</pose>
+	<inertial>
+	  <mass>10</mass>
+	</inertial>
+	<collision name="x_collision">
+	  <geometry>
+	    <box>
+	      <size>${size}</size>
+	    </box>
+	  </geometry>
+	  <surface>
+	    <contact>
+	      <collide_bitmask>0x02</collide_bitmask>
+	    </contact>
+	  </surface>
+	</collision>
+	<visual name="x_visual">
+	  <geometry>
+	    <box>
+	      <size>${size}</size>
+	    </box>
+	  </geometry>
+	  <material>
+	    <script>
+	      <uri>file://$(find imav_2017)/worlds/xacro/custom.material</uri>
+	      <name>X1</name>
+	    </script>
+	  </material>
+	</visual>
+      </link>
+    </model>
+  </xacro:macro>
 </my_macros>

Commit message: population distribution as parameter

File: worlds/xacro/imav_indoor.world.xacro (robot description, xacro)
@@ -19,17 +19,10 @@
     <xacro:wall_obstacle w_s="1.0" w_b="1.5" w_t="1.0" l_p="2.0" offset="${length1/4}" width="${width}" height="3"/>
     <xacro:wall_brand w="${length1+length2+length3}" h="${3*3}"	l="0.2" x="${length1/2+length2/2}" y="${width*2}"	z="${3*3/2}"/>
-    <xacro:poles2 h="3" r="0.25" 	w="${width*3/4}" l="${length2/2}" x="${length1/2+length2/4}"   y="${width/8}" num="10"/>
-    <xacro:trees  			w="${width*3/4}" l="${length2/2}" x="${length1/2+3*length2/4}" y="${width/8}" num="10"/>
-    <!--
-    <xacro:trees w="${width}" l="${length2/2}" x="${length1/2+3*length2/4}" y="0"/>
-    <xacro:bushes w="${width}" l="${length2/2}" x="${length1/2+3*length2/4}" y="0"/>
-    -->
+    <xacro:poles2 h="3" r="0.25" 	w="${width*3/4}" l="${length2/2}" x="${length1/2+length2/4}"   y="${width/8}" num="10" dist="uniform"/>
+    <xacro:trees  			w="${width*3/4}" l="${length2/2}" x="${length1/2+3*length2/4}" y="${width/8}" num="10" dist="uniform"/>
     <xacro:helipad_static size="1 1 0.01" x="-2.5"  y="2.5"  z="0.1"/>
     <xacro:helipad_mobile size="1 1 0.01" x="-2.5" y="-2.5" z="0.1" r="1" v="1"/>
     <xacro:QR1 size="0.5 0.5 0.01" x="${length1/2+length2+length3/2}" 	y="${width/4}"  z="0.1"/>
     <xacro:X1 size="2 2 0.01" x="${length1/2+length2+length3/2}" 	y="${-width/4}"  z="0.1"/>
-    <!--
-    <xacro:zone name="drop" 	x="${length1/2+length2+length3/2}" 	y="${-width/4}" width="2" length="2" color="${255/255}  ${0/255}  ${199/255}"/>
-    -->
   </world>
 </sdf>

File: worlds/xacro/macros.urdf.xacro (robot description, xacro)
@@ -262,5 +262,5 @@
     </link>
   </xacro:macro>
-  <xacro:macro name="poles2" params="h r w l x y num">
+  <xacro:macro name="poles2" params="h r w l x y num dist">
     <population name="pole_population">
       <model name="pole">
@@ -273,5 +273,5 @@
       <model_count>${num}</model_count>
       <distribution>
-        <type>random</type>
+        <type>${dist}</type>
       </distribution>
     </population>
@@ -296,5 +296,5 @@
     </model>
   </xacro:macro>
-  <xacro:macro name="trees" params="w l x y num">
+  <xacro:macro name="trees" params="w l x y num dist">
     <population name="tree_population">
       <model name="tree">
@@ -327,5 +327,5 @@
       <model_count>${num}</model_count>
       <distribution>
-        <type>random</type>
+        <type>${dist}</type>
       </distribution>
     </population>

Commit message: Replace the wall by a mesh

File: worlds/xacro/imav_indoor.world.xacro (robot description, xacro)
@@ -17,5 +17,6 @@
     <xacro:zone name="obstacle" 	x="${length1/2+length2/2}" 		y = "0.0" width="${width}" length="${length2}" color="${188/255} ${53/255}  ${53/255}"/>
     <xacro:zone name="target" 		x="${length1/2+length2+length3/2}" 	y = "0.0" width="${width}" length="${length3}" color="${78/255}  ${83/255}  ${199/255}"/>
-    <xacro:wall_obstacle w_s="1.0" w_b="1.5" w_t="1.0" l_p="2.0" offset="${length1/4}" width="${width}" height="3"/>
+    <!--xacro:wall_obstacle w_s="1.0" w_b="1.5" w_t="1.0" l_p="2.0" offset="${length1/4}" width="${width}" height="3"/-->
+    <xacro:wall_obstacle2 x="2.5" y="0.5"/>
     <xacro:wall_brand w="${length1+length2+length3}" h="${3*3}"	l="0.2" x="${length1/2+length2/2}" y="${width*2}"	z="${3*3/2}"/>
     <xacro:poles2 h="3" r="0.25" 	w="${width*3/4}" l="${length2/2}" x="${length1/2+length2/4}"   y="${width/8}" num="10" dist="uniform"/>

File: worlds/xacro/macros.urdf.xacro (robot description, xacro)
@@ -182,4 +182,38 @@
     </model>
   </xacro:macro>
+  <xacro:macro name="wall_obstacle2" params="x y">
+    <model name="wall2">
+      <static>1</static>
+      <pose>${x} ${y} 0 0 0 -1.5708</pose>
+        <link name="wall2_link">
+        <inertial>
+          <mass>10000</mass>
+        </inertial>
+          <visual name="visual">
+            <pose>0 0 0 0 0 0</pose>
+            <geometry>
+              <mesh>
+                <uri>file://$(find imav_2017)/worlds/xacro/wall.dae</uri>
+                <scale>0.1 0.1 0.1</scale>
+              </mesh>
+            </geometry>
+            <material>
+              <script>
+                <name>Gazebo/Wood</name>
+              </script>
+            </material>
+          </visual>
+          <collision name="collision">
+            <pose>0 0 0 0 0 0</pose>
+            <geometry>
+              <mesh>
+                <uri>file://$(find imav_2017)/worlds/xacro/wall.dae</uri>
+                <scale>0.1 0.1 0.1</scale>
+              </mesh>
+            </geometry>
+          </collision>
+        </link>
+    </model>
+  </xacro:macro>
   <xacro:macro name="box_" params="name x y z size">
     <link name='${name}'>

Commit message: Add bushes

File: worlds/xacro/imav_indoor.world.xacro (robot description, xacro)
@@ -21,4 +21,5 @@
     <xacro:poles2 h="3" r="0.25" 	w="${width*3/4}" l="${length2/2}" x="${length1/2+length2/4}"   y="${width/8}" num="10" dist="uniform"/>
     <xacro:trees  			w="${width*3/4}" l="${length2/2}" x="${length1/2+3*length2/4}" y="${width/8}" num="10" dist="uniform"/>
+    <xacro:bushes  			w="${width*3/4}" l="${length2/2}" x="${length1/2+3*length2/4}" y="${width/8}" num="6" dist="uniform"/>
     <xacro:helipad_static size="1 1 0.01" x="-2.5"  y="2.5"  z="0.1"/>
     <xacro:helipad_mobile size="1 1 0.01" x="-2.5" y="-2.5" z="0.1" r="1" v="1"/>

File: worlds/xacro/macros.urdf.xacro (robot description, xacro)
@@ -331,19 +331,36 @@
     </population>
   </xacro:macro>
-  <xacro:macro name="bushes" params="w l x y">
-    <population name="pole_population">
-      <model name="pole">
-	<include>
-          <static>true</static>
-          <uri>model://meshes/bush.dae</uri>
-        </include>
+  <xacro:macro name="bushes" params="w l x y num dist">
+    <population name="bush_population">
+      <model name="bush">
+        <static>true</static>
+        <link name="body">
+          <visual name="visual">
+            <pose>0 0 0 1.5708 0 0</pose>
+            <geometry>
+              <mesh>
+                <uri>file://$(find imav_2017)/worlds/xacro/tree1.dae</uri>
+                <scale>0.01 0.004 0.01</scale>
+              </mesh>
+            </geometry>
+          </visual>
+          <collision name="collision">
+            <pose>0 0 0 1.5708 0 0</pose>
+            <geometry>
+              <mesh>
+                <uri>file://$(find imav_2017)/worlds/xacro/tree1.dae</uri>
+                <scale>0.01 0.004 0.01</scale>
+              </mesh>
+            </geometry>
+          </collision>
+        </link>
       </model>
-      <pose>${x} ${y} 0 0 0 0</pose>
+      <pose>${x} ${y} -0.5 0 0 0</pose>
       <box>
         <size>${l} ${w} 0.1</size>
       </box>
-      <model_count>10</model_count>
+      <model_count>${num}</model_count>
       <distribution>
-        <type>uniform</type>
+        <type>${dist}</type>
       </distribution>
     </population>
