Commit message: add more walls and textures

File: worlds/xacro/imav_indoor.world.xacro (robot description, xacro)
@@ -2,8 +2,8 @@
 <sdf version='1.6'>
   <world name="imav_world" xmlns:xacro="http://www.ros.org/wiki/xacro">
-    <xacro:property name="width" value="13" />
+    <xacro:property name="width" value="10" />
     <xacro:property name="length1" value="10" />
     <xacro:property name="length2" value="10" />
-    <xacro:property name="length3" value="13" />
+    <xacro:property name="length3" value="7" />
     <xacro:include filename="$(find imav_2017)/worlds/xacro/macros.urdf.xacro" />
     <xacro:light_source/>
@@ -14,12 +14,16 @@
     <xacro:scn amb="0.4 0.4 0.4 1" backg="${53/255} ${147/255} ${37/255} 1"/>
     -->
-    <xacro:zone name="takoff_landing" x="0"                              y="0.0" width="${width}" length="${length1}" color="${22/255}  ${176/255} ${37/255}"/>
+    <!--xacro:zone name="takoff_landing" x="0"                              y="0.0" width="${width}" length="${length1}" color="${22/255}  ${176/255} ${37/255}"/>
     <xacro:zone name="obstacle"       x="${length1/2+length2/2}"         y="0.0" width="${width}" length="${length2}" color="${188/255} ${53/255}  ${53/255}"/>
-    <xacro:zone name="target"         x="${length1/2+length2+length3/2}" y="0.0" width="${width}" length="${length3}" color="${78/255}  ${83/255}  ${199/255}"/>
+    <xacro:zone name="target"         x="${length1/2+length2+length3/2}" y="0.0" width="${width}" length="${length3}" color="${78/255}  ${83/255}  ${199/255}"/-->
+    <xacro:zone_texture name="takoff_landing" x="0"                              y="0.0" width="${width}" length="${length1}" texture="Kitchen/WoodFloor"/>
+    <xacro:zone_texture name="obstacle"       x="${length1/2+length2/2}"         y="0.0" width="${width}" length="${length2}" texture="Kitchen/Grass"/>
+    <xacro:zone_texture name="target"         x="${length1/2+length2+length3/2}" y="0.0" width="${width}" length="${length3}" texture="Kitchen/CounterTop"/>
     <!--
     <xacro:wall_obstacle w_s="1.0" w_b="1.5" w_t="1.0" l_p="2.0" offset="${length1/4}" width="${width}" height="3"/>
     -->
     <xacro:wall_obstacle2 x="2.5" y="0.5"/>
-    <xacro:wall_brand w="${length1+length2+length3}" h="${3*3}" l="0.2" x="${length1/2+length2/2}" y="${width*2}" z="${3*3/2}"/>
+    <xacro:wall_brand w="${length1+length2+length3}" h="${width/2}" l="0.2" x="${length1/2+length2/2-length3/4}" y="${width}" z="${width/4}"/>
+    <xacro:wall_imav w="${width}" h="${width/2}" l="0.2" x="${length1/2+length2+length3}" y="0" z="${width/4}"/>
     <xacro:poles2 w="${width*3/4}" l="${length2/2}" x="${length1/2+length2/4}"   y="${width/8}" num="10" dist="uniform" h="3" r="0.25"/>
     <xacro:trees  w="${width*3/4}" l="${length2/2}" x="${length1/2+3*length2/4}" y="${width/8}" num="10" dist="uniform"/>

File: worlds/xacro/macros.urdf.xacro (robot description, xacro)
@@ -49,4 +49,54 @@
     </model>
   </xacro:macro>
+  <xacro:macro name="zone_texture" params="name width length texture x y">
+    <model name="${name}_zone">
+      <static>1</static>
+      <pose>${x} ${y} 0 0 0 0</pose>
+      <link name='link'>
+        <collision name='collision'>
+          <geometry>
+            <plane>
+              <normal>0 0 1</normal>
+              <size>${length} ${width}</size>
+            </plane>
+          </geometry>
+          <surface>
+            <friction>
+              <ode>
+                <mu>100</mu>
+                <mu2>50</mu2>
+              </ode>
+            </friction>
+            <bounce/>
+            <contact>
+              <ode/>
+            </contact>
+          </surface>
+          <max_contacts>10</max_contacts>
+        </collision>
+        <visual name='visual'>
+          <cast_shadows>0</cast_shadows>
+          <geometry>
+            <plane>
+              <normal>0 0 1</normal>
+              <size>${length} ${width}</size>
+            </plane>
+          </geometry>
+          <material>
+            <script>
+              <name>${texture}</name>
+            </script>
+          </material>
+        </visual>
+        <velocity_decay>
+          <linear>0</linear>
+          <angular>0</angular>
+        </velocity_decay>
+        <self_collide>0</self_collide>
+        <kinematic>0</kinematic>
+        <gravity>1</gravity>
+      </link>
+    </model>
+  </xacro:macro>
   <xacro:macro name="light_source">
     <light name="sun" type="directional">
@@ -151,4 +201,40 @@
               <uri>file://$(find imav_2017)/worlds/xacro/custom.material</uri>
               <name>MathWorks_branding</name>
+            </script>
+          </material>
+        </visual>
+      </link>
+    </model>
+  </xacro:macro>
+  <xacro:macro name="wall_imav" params="w h l x y z">
+    <model name="branded_wall">
+      <static>true</static>
+      <pose>${x} ${y} ${z} 0 0 -1.5708</pose>
+      <link name="wall_link">
+        <inertial>
+          <mass>10000</mass>
+        </inertial>
+        <collision name="wall_imav_collision">
+          <geometry>
+            <box>
+              <size>${w} ${l} ${h}</size>
+            </box>
+          </geometry>
+          <surface>
+            <contact>
+              <collide_bitmask>0x02</collide_bitmask>
+            </contact>
+          </surface>
+        </collision>
+        <visual name="wall_imav_visual">
+          <geometry>
+            <box>
+              <size>${w} ${l} ${h}</size>
+            </box>
+          </geometry>
+          <material>
+            <script>
+              <uri>file://$(find imav_2017)/worlds/xacro/custom.material</uri>
+              <name>imav_branding</name>
             </script>
           </material>
